File: watch-power.kicad_pcb (KiCad board)
At the start: 2 copper layers, 30 x 22 mm, 21 parts, among them IC1 BQ24230, IC2 LC709203FQH-01TWG, IC3 DRV2603RUNR, IC4 TPS63030, J1 47346-0001, J2 1-1734592-4, M1 Vibramotor

Commit message: big save
Parts:
- added AC1: LSM6DSOXTR, LSM6DSOXTR:LGA-14_1, F.Cu at (142.0, 16.6)
- added ANT1: 2450AT18B100E, 2450AT18B100E:ANTC3216X140N, F.Cu at (131.6, 54.0)
- added C10: 1.0uF, Capacitor_SMD:C_0603_1608Metric, F.Cu at (113.0, 45.8)
- added C11: 100nF, Capacitor_SMD:C_0402_1005Metric, F.Cu at (104.6, 58.8)
- added C12: 2.7pF, Capacitor_SMD:C_0402_1005Metric, F.Cu at (123.3, 54.1)
- added C13: 12pF, Capacitor_SMD:C_0402_1005Metric, F.Cu at (93.4, 41.4)
- added C14: 100pF, Capacitor_SMD:C_0402_1005Metric, F.Cu at (120.8, 47.8)
- added C15: 4.7uF, Capacitor_SMD:C_0603_1608Metric, F.Cu at (104.2, 55.8)
- added C17: 100nF, Capacitor_SMD:C_0402_1005Metric, F.Cu at (109.3, 50.9)
- added C23: 12pF, Capacitor_SMD:C_0402_1005Metric, F.Cu at (103.3, 35.0)
- added C24: 12pF, Capacitor_SMD:C_0402_1005Metric, F.Cu at (96.4, 40.0)
- added C8: 0.8pF, Capacitor_SMD:C_0402_1005Metric, F.Cu at (119.0, 53.5)
- added C9: 12pF, Capacitor_SMD:C_0402_1005Metric, F.Cu at (100.9, 33.0)
- added IC2: MMBT2222ALT1G, MMBT2222ALT1G:SOT96P237X111-3N, F.Cu at (135.9, -10.0)
- added L2: HK100515NJ-T, HK100515NJ-T:INDC1005X55N, F.Cu at (116.0, 72.3)
- added L3: LBMF1608T100K, LBMF1608T100K:INDC1608X100N, F.Cu at (115.5, 69.1)
- added L4: LQP15MN1N8B02D, LQP15MN1N8B02D:LQP15MN10NG02D, F.Cu at (127.1, 54.2)
- added L5: LQP15MN2N7B02D, LQP15MN1N8B02D:LQP15MN10NG02D, F.Cu at (123.8, 52.3)
- added L6: LQP15MN3N9B02D, LQP15MN1N8B02D:LQP15MN10NG02D, F.Cu at (121.0, 54.0)
- added Q1: 2N2219, Package_TO_SOT_THT:TO-39-3, F.Cu at (111.0, -24.3)
- added R8: 100k, Resistor_SMD:R_0603_1608Metric, F.Cu at (46.4, 57.7)
- added R9: 100k, Resistor_SMD:R_0603_1608Metric, F.Cu at (50.4, 57.7)
- added U1: nRF52832-QFxx, Package_DFN_QFN:QFN-48-1EP_6x6mm_P0.4mm_EP4.6x4.6mm, F.Cu at (114.2, 53.6)
- added U2: APDS9960, APDS-9960:APDS-9950, F.Cu at (141.1, 23.5)
- added U3: ST7735, ST7735:ST7735_curved, F.Cu at (136.4, -20.6)
- moved R1 0.48 mm to (33.1, 39.9)
Connections:
- net Net-(C5-Pad1) renamed BATT_P
- C1 pad 2: Net-(C1-Pad2) -> BATT_M
- C3 pad 2: Net-(C3-Pad2) -> BATT_M
- C4 pad 1: Net-(C4-Pad1) -> +3V3
- C4 pad 2: Net-(C4-Pad2) -> BATT_M
- C5 pad 2: Net-(C5-Pad2) -> BATT_M
- C6 pad 1: Net-(C6-Pad1) -> +3V3
- C6 pad 2: Net-(C6-Pad2) -> BATT_M
- C7 pad 2: Net-(C7-Pad2) -> BATT_M
- J1 pad 1: Net-(J1-Pad1) -> Net-(C1-Pad1)
- J1 pad 5: Net-(J1-Pad5) -> BATT_M
- L1 pad 1: Net-(L1-Pad1) -> Net-(IC1-Pad4)
- L1 pad 2: Net-(L1-Pad2) -> Net-(IC1-Pad2)
- R1 pad 1: Net-(R1-Pad1) -> BATT_M
- R3 pad 1: Net-(R3-Pad1) -> BATT_M
- R4 pad 1: Net-(R4-Pad1) -> Net-(C3-Pad1)
- R4 pad 2: Net-(R4-Pad2) -> Net-(IC1-Pad10)
- R5 pad 1: Net-(R5-Pad1) -> Net-(IC1-Pad10)
- R5 pad 2: Net-(R5-Pad2) -> BATT_M

Commit message: big save
Parts:
- moved U3 67.0 mm to (84.0, 21.2)
- moved L2 55.1 mm to (73.9, 36.6), turned to 270 degrees
- moved IC2 53.2 mm to (86.1, 8.64)
- moved L3 49.7 mm to (75.1, 40.1), turned to 270 degrees
- moved C17 37.9 mm to (72.2, 43.4)
- moved C10 37.8 mm to (76.3, 36.7), turned to 90 degrees
- moved L6 37.7 mm to (84.2, 46.0)
- moved ANT1 37.7 mm to (94.8, 46.0)
- moved C12 37.7 mm to (86.5, 46.1)
- moved C8 37.7 mm to (82.2, 45.5)
- moved L4 37.7 mm to (90.3, 46.2)
- moved L5 37.7 mm to (87.0, 44.3)
- moved U1 37.7 mm to (77.3, 45.6)
- moved C14 37.7 mm to (83.4, 42.7)
- moved C9 35.7 mm to (68.8, 48.6), turned to 180 degrees
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
Commit message: save
Parts:
- added C18: 100nF, Capacitor_SMD:C_0402_1005Metric, F.Cu at (93.6, 44.0)
- added C19: 100nF, Capacitor_SMD:C_0402_1005Metric, F.Cu at (91.4, 43.8)
- added C20: 0.1uF, Capacitor_SMD:C_0201_0603Metric, F.Cu at (33.1, 57.7)
- added C21: 1uF, Capacitor_SMD:C_0402_1005Metric, F.Cu at (78.9, 50.9)
- added C22: 1uF, Capacitor_SMD:C_0402_1005Metric, F.Cu at (78.9, 48.5)
- added C25: 100nF, Capacitor_SMD:C_0402_1005Metric, F.Cu at (82.5, 39.8)
- added R10: 1k, Resistor_SMD:R_0402_1005Metric, F.Cu at (86.1, 39.6)
- added R11: 10k, Resistor_SMD:R_0402_1005Metric, F.Cu at (84.2, 39.8)
- added R13: 10k, Resistor_SMD:R_0402_1005Metric, F.Cu at (82.5, 46.6)
- added R15: 10k, Resistor_SMD:R_0402_1005Metric, F.Cu at (83.6, 45.2)
- added R17: 100R, Resistor_SMD:R_0402_1005Metric, F.Cu at (82.5, 37.5)
- added R6: 22R, Resistor_SMD:R_0402_1005Metric, F.Cu at (77.2, 48.6)
- added R7: 10k, Resistor_SMD:R_0402_1005Metric, F.Cu at (85.6, 49.4)
- ANT1, C10, C11, C12, C13, C14, C15, C17, C23, C24, C8, C9, L2, L3, L4, L5, L6, U1: moved to B.Cu
- moved U2 36.4 mm to (81.5, 49.9)
- moved L2 34.0 mm to (71.1, 70.5), turned to 90 degrees
- moved C10 33.8 mm to (73.5, 70.4), turned to 270 degrees
- moved AC1 32.4 mm to (88.6, 43.8), turned to 90 degrees
- moved IC2 28.0 mm to (85.3, 36.6), turned to 180 degrees
- moved L3 26.9 mm to (72.3, 66.9), turned to 90 degrees
- moved C24 26.4 mm to (83.7, 66.7), turned to 90 degrees
- moved C23 26.4 mm to (80.5, 66.7), turned to 270 degrees
- moved C15 22.9 mm to (68.9, 64.9)
- moved C14 21.9 mm to (80.6, 64.4)
- moved C17 20.4 mm to (69.4, 63.6)
- moved U3 20.0 mm to (81.5, 41.0), turned to 180 degrees
- moved L5 18.7 mm to (84.2, 62.8), turned to 90 degrees
- moved C8 16.4 mm to (79.4, 61.6), turned to 270 degrees
- moved U1 16.1 mm to (74.5, 61.5)
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Connections:
- IC2 pad 2: Net-(IC2-Pad2) -> BATT_M
- U3 pad 11: LEDK -> Net-(R17-Pad1)
Other:
- board size 30 x 22 mm -> 68 x 22 mm
- board text added: "0201-es ellenállás?? sztem legyen csak 0402"

Commit message: add piezo
Parts:
- added Q1: BC847, Package_TO_SOT_SMD:SOT-23, F.Cu at (53.6, 50.8)
- added R18: 1k, Resistor_SMD:R_0603_1608Metric, F.Cu at (58.5, 50.4)
Connections:
- LS1 pad 1: Net-(LS1-Pad1) -> +3V3

Commit message: save before drastic rearranger
Parts:
- moved Q1 54.4 mm to (82.3, 22.0)
